Commit message: feat: created a package for custom gazebo world

File: src/carter_description/urdf/carter.urdf.xacro (robot description, xacro)
@@ -11,5 +11,5 @@
          </geometry>
          <material name="chassis_material">
-            <color rgba="0.5 0.5 0.5 1.0" />
+            <color rgba="0.5 0.5 0.5 0.9" />
          </material>
       </visual>
@@ -33,5 +33,5 @@
          </geometry>
          <material name="wheel_material">
-            <color rgba="0.5 0.5 0.5 0.8" />
+            <color rgba="0 0 0 0.9" />
          </material>
       </visual>
@@ -55,5 +55,5 @@
          </geometry>
          <material name="wheel_material">
-            <color rgba="0.5 0.5 0.5 0.8" />
+            <color rgba="0 0 0  0.9" />
          </material>
       </visual>

File: src/carter_description/urdf/lidar.xacro (robot description, xacro)
@@ -4,5 +4,5 @@
   <link name="lidar_link">
     <visual>
-      <origin xyz="-0.05 0 0.42" rpy="0 0 0"/>
+      <origin xyz="-0.0 0 0.0" rpy="0 0 0"/>
       <geometry>
         <cylinder radius="0.01" length="0.01" />
@@ -24,10 +24,10 @@
     <parent link="chassis_link"/>
     <child link="lidar_link"/>
-    <origin rpy="0 0 0.42" xyz="0 0 0" />
+    <origin rpy="0 0 0" xyz="-0.05 0 0.42" />
   </joint>
   <gazebo reference="lidar_link">
-    <sensor name="lidar" type='gpu_lidar'>
+    <sensor name="scan" type='gpu_lidar'>
       <pose>0 0 0.2 0 0 0</pose>
-      <topic>lidar</topic>
+      <topic>scan</topic>
       <update_rate>10</update_rate>
       <ray>
